File: r1/src/_audio.kicad_sch (KiCad schematic)
At the start: 24 parts, among them J10 PJ-320D, U7 PAM8908, U8 PCM5100A

Commit message: Update all symbols
Connections:
- net +3.3V: no longer U7.6 (G0)
- net GND: no longer U7.7 (G1)
- new net AMP_GAIN0: U7.6 (G0)
- new net AMP_GAIN1: U7.7 (G1)
Changed lines of the file:
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@@
+    (stroke (width 0) (type default))
+  )
+  (wire (pts (xy 160.02 113.03) (xy 167.64 113.03))
     (stroke (width 0) (type default))
   )
@@
   )
   (wire (pts (xy 193.04 107.95) (xy 195.58 107.95))
+    (stroke (width 0) (type default))
+  )
+  (wire (pts (xy 160.02 110.49) (xy 167.64 110.49))
     (stroke (width 0) (type default))
   )
@@
     (effects (font (size 1.27 1.27)) (justify right))
   )
+  (hierarchical_label "AMP_GAIN1" (shape input) (at 160.02 113.03 180) (fields_autoplaced)
+    (effects (font (size 1.27 1.27)) (justify right))
+  )
   (hierarchical_label "I2S_SD" (shape input) (at 69.85 85.09 180)
     (effects (font (size 1.27 1.27)) (justify right))
   )
   (hierarchical_label "I2S_WS" (shape input) (at 69.85 82.55 180)
+    (effects (font (size 1.27 1.27)) (justify right))
+  )
+  (hierarchical_label "AMP_GAIN0" (shape input) (at 160.02 110.49 180) (fields_autoplaced)
     (effects (font (size 1.27 1.27)) (justify right))
   )
@@
         )
       )
-    )
-  )
-  (symbol (lib_id "power:+3.3V") (at 167.64 110.49 90) (unit 1)
-    (in_bom yes) (on_board yes) (dnp no)
-    (property "Reference" "#PWR080" (at 171.45 110.49 0)
-      (effects (font (size 1.27 1.27)) hide)
-    )
-    (property "Value" "+3.3V" (at 161.29 110.49 90)
-      (effects (font (size 1.27 1.27)))
-    )
-    (property "Footprint" "" (at 167.64 110.49 0)
-      (effects (font (size 1.27 1.27)) hide)
-    )
-    (property "Datasheet" "" (at 167.64 110.49 0)
-      (effects (font (size 1.27 1.27)) hide)
-    )
-    (pin "1")
-    (instances
-      (project "tr23-badge-r1"
-        (path "/ab725fe7-4504-40ef-b6af-82d065d00fb6/00000000-0000-0000-0000-00005dd6a7f2"
-          (reference "#PWR080") (unit 1)
-        )
-      )
-    )
-  )
-  (symbol (lib_id "power:GND") (at 167.64 113.03 270) (unit 1)
-    (in_bom yes) (on_board yes) (dnp no)
-    (property "Reference" "#PWR081" (at 161.29 113.03 0)
-      (effects (font (size 1.27 1.27)) hide)
-    )
-    (property "Value" "GND" (at 162.56 113.03 90)
-      (effects (font (size 1.27 1.27)))
-    )
-    (property "Footprint" "" (at 167.64 113.03 0)
-      (effects (font (size 1.27 1.27)) hide)
-    )
-    (property "Datasheet" "" (at 167.64 113.03 0)
-      (effects (font (size 1.27 1.27)) hide)
-    )
-    (pin "1")
-    (instances
-      (project "tr23-badge-r1"
-        (path "/ab725fe7-4504-40ef-b6af-82d065d00fb6/00000000-0000-0000-0000-00005dd6a7f2"
-          (reference "#PWR081") (unit 1)
-        )
-      )
