File: r1/src/_display.kicad_sch (KiCad schematic)
At the start: 3 parts, among them J5 AFC07-S40ECA-00, Q6 AP2302B

Commit message: Reannotate component refs
Parts:
- renumbered J5 to J4
Changed lines of the file:
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@@
   (symbol (lib_id "power:GND") (at 147.32 156.21 0) (unit 1)
     (in_bom yes) (on_board yes) (dnp no) (fields_autoplaced)
-    (property "Reference" "#PWR054" (at 147.32 162.56 0)
+    (property "Reference" "#PWR043" (at 147.32 162.56 0)
       (effects (font (size 1.27 1.27)) hide)
     )
@@
       (project "tr23-badge-r1"
         (path "/ab725fe7-4504-40ef-b6af-82d065d00fb6/00000000-0000-0000-0000-00005e536877"
-          (reference "#PWR054") (unit 1)
+          (reference "#PWR043") (unit 1)
         )
       )
@@
         )
         (path "/ab725fe7-4504-40ef-b6af-82d065d00fb6/00000000-0000-0000-0000-00005e536877"
-          (reference "R21") (unit 1)
+          (reference "R20") (unit 1)
         )
       )
@@
   (symbol (lib_id "power:GND") (at 119.38 156.21 0) (unit 1)
     (in_bom yes) (on_board yes) (dnp no) (fields_autoplaced)
-    (property "Reference" "#PWR057" (at 119.38 162.56 0)
+    (property "Reference" "#PWR040" (at 119.38 162.56 0)
       (effects (font (size 1.27 1.27)) hide)
     )
@@
       (project "tr23-badge-r1"
         (path "/ab725fe7-4504-40ef-b6af-82d065d00fb6/00000000-0000-0000-0000-00005e536877"
-          (reference "#PWR057") (unit 1)
+          (reference "#PWR040") (unit 1)
         )
       )
@@
         )
         (path "/ab725fe7-4504-40ef-b6af-82d065d00fb6/00000000-0000-0000-0000-00005e536877"
-          (reference "#PWR056") (unit 1)
+          (reference "#PWR042") (unit 1)
         )
       )
@@
   (symbol (lib_id "power:GND") (at 129.54 156.21 0) (unit 1)
     (in_bom yes) (on_board yes) (dnp no) (fields_autoplaced)
-    (property "Reference" "#PWR055" (at 129.54 162.56 0)
+    (property "Reference" "#PWR041" (at 129.54 162.56 0)
       (effects (font (size 1.27 1.27)) hide)
     )
@@
       (project "tr23-badge-r1"
         (path "/ab725fe7-4504-40ef-b6af-82d065d00fb6/00000000-0000-0000-0000-00005e536877"
-          (reference "#PWR055") (unit 1)
+          (reference "#PWR041") (unit 1)
         )
       )
@@
   (symbol (lib_id "Connector_Generic_MountingPin:Conn_01x40_MountingPin") (at 158.75 99.06 0) (unit 1)
     (in_bom yes) (on_board yes) (dnp no)
-    (property "Reference" "J5" (at 157.48 44.45 0)
+    (property "Reference" "J4" (at 157.48 44.45 0)
       (effects (font (size 1.27 1.27)) (justify left))
     )
@@
       (project "tr23-badge-r1"
         (path "/ab725fe7-4504-40ef-b6af-82d065d00fb6/00000000-0000-0000-0000-00005e536877"
-          (reference "J5") (unit 1)
+          (reference "J4") (unit 1)
         )
       )
@@
   (symbol (lib_id "power:GND") (at 158.75 154.94 0) (unit 1)
     (in_bom yes) (on_board yes) (dnp no) (fields_autoplaced)
-    (property "Reference" "#PWR058" (at 158.75 161.29 0)
+    (property "Reference" "#PWR044" (at 158.75 161.29 0)
       (effects (font (size 1.27 1.27)) hide)
     )
@@
       (project "tr23-badge-r1"
         (path "/ab725fe7-4504-40ef-b6af-82d065d00fb6/00000000-0000-0000-0000-00005e536877"
-          (reference "#PWR058") (unit 1)
-        )
-      )
+          (reference "#PWR044") (unit 1)
+        )
+      )

Commit message: Assign footprints from jeffmakes-footprints lib
Parts:
- J4: footprint (none) -> jeffmakes_footprints:D-1206
- Q6: footprint (none) -> jeffmakes_footprints:USB-A-short-body-in-cutout-type-strenghening-vias
Changed lines of the file:
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@@
       (effects (font (size 1.27 1.27)) (justify left))
     )
-    (property "Footprint" "" (at 132.08 143.51 0)
+    (property "Footprint" "jeffmakes_footprints:USB-A-short-body-in-cutout-type-strenghening-vias" (at 132.08 143.51 0)
       (effects (font (size 1.27 1.27)) hide)
     )
@@
       (effects (font (size 1.27 1.27)) (justify left))
     )
-    (property "Footprint" "" (at 158.75 99.06 0)
+    (property "Footprint" "jeffmakes_footprints:D-1206" (at 158.75 99.06 0)
       (effects (font (size 1.27 1.27)) hide)
     )
