File: r1/src/_radio.kicad_sch (KiCad schematic)
At the start: 49 parts, among them J8 DNP, U9 CC1200, Y2 40Mhz

Commit message: ERC pass. Schematic complete.
Parts:
- AE1: footprint jeffmakes_footprints:Antenna_TI_DN038 -> jeffmakes-footprints:Antenna_TI_DN038
Changed lines of the file:
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@@
       (effects (font (size 1.27 1.27)) (justify left))
     )
-    (property "Footprint" "jeffmakes_footprints:Antenna_TI_DN038" (at 222.25 123.19 0)
+    (property "Footprint" "jeffmakes-footprints:Antenna_TI_DN038" (at 222.25 123.19 0)
       (effects (font (size 1.27 1.27)) hide)
     )

Commit message: Assign footprints
Parts:
- AE1: footprint jeffmakes-footprints:Antenna_TI_DN038 -> jeffmakes_footprints:Antenna_TI_DN038
Changed lines of the file:
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@@
       (effects (font (size 1.27 1.27)) (justify left))
     )
-    (property "Footprint" "jeffmakes-footprints:Antenna_TI_DN038" (at 222.25 123.19 0)
+    (property "Footprint" "jeffmakes_footprints:Antenna_TI_DN038" (at 222.25 123.19 0)
       (effects (font (size 1.27 1.27)) hide)
     )
