File: r1/src/_radio.kicad_sch (KiCad schematic)
At the start: 49 parts, among them J8 DNP, U9 CC1200, Y2 40Mhz

Commit message: Assign more net classes. Set RF 50ohm width with coplanar ground-backed calculation
Parts:
- J8: footprint Connector_Coaxial:SMA_Amphenol_132291-12_Vertical -> Connector_Coaxial:SMA_Amphenol_132134-10_Vertical
Connections:
- net ANT_EXT: now reaches J8.1 (In), R30.1
- net ANT: now reaches AE1.1 (A), C69.2, L9.2
Other:
- moved on the sheet: AE1, J8, TP34, TP35
Changed lines of the file:
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@@
+    (stroke (width 0) (type default))
+  )
+  (wire (pts (xy 189.23 146.685) (xy 189.23 143.51))
     (stroke (width 0) (type default))
   )
@@
     (stroke (width 0) (type default))
   )
+  (wire (pts (xy 73.66 71.12) (xy 74.93 71.12))
+    (stroke (width 0) (type default))
+  )
   (wire (pts (xy 170.18 81.28) (xy 170.18 85.09))
     (stroke (width 0) (type default))
@@
     (stroke (width 0) (type default))
   )
+  (wire (pts (xy 73.66 68.58) (xy 74.93 68.58))
+    (stroke (width 0) (type default))
+  )
   (wire (pts (xy 200.66 48.26) (xy 210.82 48.26))
     (stroke (width 0) (type default))
@@
     (stroke (width 0) (type default))
   )
-  (wire (pts (xy 67.31 68.58) (xy 53.34 68.58))
+  (wire (pts (xy 66.675 68.58) (xy 53.34 68.58))
     (stroke (width 0) (type default))
   )
@@
     (stroke (width 0) (type default))
   )
-  (wire (pts (xy 222.25 133.35) (xy 222.25 128.27))
+  (wire (pts (xy 227.965 133.35) (xy 227.965 128.27))
     (stroke (width 0) (type default))
   )
@@
     (stroke (width 0) (type default))
   )
-  (wire (pts (xy 67.31 76.2) (xy 74.93 76.2))
+  (wire (pts (xy 66.675 76.2) (xy 74.93 76.2))
     (stroke (width 0) (type default))
   )
@@
     (stroke (width 0) (type default))
   )
-  (wire (pts (xy 218.44 133.35) (xy 222.25 133.35))
+  (wire (pts (xy 218.44 133.35) (xy 227.965 133.35))
     (stroke (width 0) (type default))
   )
@@
     (stroke (width 0) (type default))
   )
-  (wire (pts (xy 67.31 76.2) (xy 67.31 68.58))
+  (wire (pts (xy 66.675 76.2) (xy 66.675 68.58))
     (stroke (width 0) (type default))
   )
@@
   (wire (pts (xy 184.15 133.35) (xy 189.23 133.35))
     (stroke (width 0) (type default))
+  )
+  (label "ANT" (at 220.345 133.35 0) (fields_autoplaced)
+    (effects (font (size 1.27 1.27)) (justify left bottom))
+  )
+  (label "ANT_EXT" (at 189.23 146.05 0) (fields_autoplaced)
+    (effects (font (size 1.27 1.27)) (justify left bottom))
   )
   (hierarchical_label "~{RESET}" (shape input) (at 62.23 48.26 180) (fields_autoplaced)
@@
   (hierarchical_label "~{CS}" (shape input) (at 62.23 53.34 180) (fields_autoplaced)
     (effects (font (size 1.27 1.27)) (justify right))
+  )
+  (netclass_flag "" (length 1.27) (shape dot) (at 151.13 142.24 270) (fields_autoplaced)
+    (effects (font (size 1.27 1.27)) (justify right bottom))
+    (property "Netclass" "RF_50_ohm" (at 152.4 141.6304 90)
+      (effects (font (size 1.27 1.27) italic) (justify left) hide)
+    )
+  )
+  (netclass_flag "" (length 1.27) (shape dot) (at 121.92 133.35 0) (fields_autoplaced)
+    (effects (font (size 1.27 1.27)) (justify left bottom))
+    (property "Netclass" "RF_50_ohm" (at 122.5296 132.08 0)
+      (effects (font (size 1.27 1.27) italic) (justify left))
+    )
+  )
+  (netclass_flag "" (length 1.27) (shape dot) (at 202.565 133.35 0) (fields_autoplaced)
+    (effects (font (size 1.27 1.27)) (justify left bottom))
+    (property "Netclass" "RF_50_ohm" (at 203.1746 132.08 0)
+      (effects (font (size 1.27 1.27) italic) (justify left) hide)
+    )
+  )
+  (netclass_flag "" (length 1.27) (shape dot) (at 140.97 142.24 90) (fields_autoplaced)
+    (effects (font (size 1.27 1.27)) (justify left bottom))
+    (property "Netclass" "RF_50_ohm" (at 139.7 141.6304 90)
+      (effects (font (size 1.27 1.27) italic) (justify left) hide)
+    )
+  )
+  (netclass_flag "" (length 1.27) (shape dot) (at 186.69 133.35 0) (fields_autoplaced)
+    (effects (font (size 1.27 1.27)) (justify left bottom))
+    (property "Netclass" "RF_50_ohm" (at 187.2996 132.08 0)
+      (effects (font (size 1.27 1.27) italic) (justify left) hide)
+    )
+  )
+  (netclass_flag "" (length 1.27) (shape dot) (at 164.465 133.35 0) (fields_autoplaced)
+    (effects (font (size 1.27 1.27)) (justify left bottom))
+    (property "Netclass" "RF_50_ohm" (at 165.0746 132.08 0)
+      (effects (font (size 1.27 1.27) italic) (justify left) hide)
+    )
   )
   (symbol (lib_id "Device:C") (at 129.54 53.34 0) (unit 1)
@@
     )
   )
-  (symbol (lib_id "Connector:TestPoint") (at 74.93 68.58 90) (unit 1)
-    (in_bom yes) (on_board yes) (dnp no)
-    (property "Reference" "TP34" (at 73.1012 65.9638 90)
-      (effects (font (size 1.27 1.27)))
-    )
-    (property "Value" "~" (at 73.1012 65.9384 90)
-      (effects (font (size 1.27 1.27)))
-    )
-    (property "Footprint" "TestPoint:TestPoint_Pad_D1.0mm" (at 74.93 63.5 0)
-      (effects (font (size 1.27 1.27)) hide)
-    )
-    (property "Datasheet" "~" (at 74.93 63.5 0)
+  (symbol (lib_id "Connector:TestPoint") (at 73.66 68.58 90) (unit 1)
+    (in_bom yes) (on_board yes) (dnp no)
+    (property "Reference" "TP34" (at 71.12 66.675 90)
+      (effects (font (size 1.27 1.27)))
+    )
+    (property "Value" "~" (at 71.8312 65.9384 90)
+      (effects (font (size 1.27 1.27)))
+    )
+    (property "Footprint" "TestPoint:TestPoint_Pad_D1.0mm" (at 73.66 63.5 0)
+      (effects (font (size 1.27 1.27)) hide)
+    )
+    (property "Datasheet" "~" (at 73.66 63.5 0)
       (effects (font (size 1.27 1.27)) hide)
     )
@@
     )
   )
-  (symbol (lib_id "Connector:TestPoint") (at 74.93 71.12 90) (unit 1)
-    (in_bom yes) (on_board yes) (dnp no)
-    (property "Reference" "TP35" (at 73.1012 68.5038 90)
-      (effects (font (size 1.27 1.27)))
-    )
-    (property "Value" "~" (at 73.1012 68.4784 90)
-      (effects (font (size 1.27 1.27)))
-    )
-    (property "Footprint" "TestPoint:TestPoint_Pad_D1.0mm" (at 74.93 66.04 0)
-      (effects (font (size 1.27 1.27)) hide)
-    )
-    (property "Datasheet" "~" (at 74.93 66.04 0)
+  (symbol (lib_id "Connector:TestPoint") (at 73.66 71.12 90) (unit 1)
+    (in_bom yes) (on_board yes) (dnp no)
+    (property "Reference" "TP35" (at 71.12 69.215 90)
+      (effects (font (size 1.27 1.27)))
+    )
+    (property "Value" "~" (at 71.8312 68.4784 90)
+      (effects (font (size 1.27 1.27)))
+    )
+    (property "Footprint" "TestPoint:TestPoint_Pad_D1.0mm" (at 73.66 66.04 0)
+      (effects (font (size 1.27 1.27)) hide)
+    )
+    (property "Datasheet" "~" (at 73.66 66.04 0)
       (effects (font (size 1.27 1.27)) hide)
     )
@@
     )
   )
-  (symbol (lib_id "Connector:Conn_Coaxial") (at 189.23 148.59 270) (unit 1)
-    (in_bom yes) (on_board yes) (dnp no)
-    (property "Reference" "J8" (at 191.77 145.5928 90)
-      (effects (font (size 1.27 1.27)) (justify left))
-    )
-    (property "Value" "DNP" (at 191.77 147.9042 90)
-      (effects (font (size 1.27 1.27)) (justify left))
-    )
-    (property "Footprint" "Connector_Coaxial:SMA_Amphenol_132291-12_Vertical" (at 189.23 148.59 0)
-      (effects (font (size 1.27 1.27)) hide)
-    )
-    (property "Datasheet" " ~" (at 189.23 148.59 0)
+  (symbol (lib_id "Connector:Conn_Coaxial") (at 189.23 151.765 270) (unit 1)
+    (in_bom yes) (on_board yes) (dnp no)
+    (property "Reference" "J8" (at 191.77 148.7678 90)
+      (effects (font (size 1.27 1.27)) (justify left))
+    )
+    (property "Value" "DNP" (at 191.77 151.0792 90)
+      (effects (font (size 1.27 1.27)) (justify left))
+    )
+    (property "Footprint" "Connector_Coaxial:SMA_Amphenol_132134-10_Vertical" (at 189.23 151.765 0)
+      (effects (font (size 1.27 1.27)) hide)
+    )
+    (property "Datasheet" " ~" (at 189.23 151.765 0)
       (effects (font (size 1.27 1.27)) hide)
     )
@@
     )
   )
-  (symbol (lib_id "power:GND") (at 184.15 148.59 270) (unit 1)
-    (in_bom yes) (on_board yes) (dnp no)
-    (property "Reference" "#PWR0146" (at 177.8 148.59 0)
-      (effects (font (size 1.27 1.27)) hide)
-    )
-    (property "Value" "GND" (at 180.8988 148.717 90)
+  (symbol (lib_id "power:GND") (at 184.15 151.765 270) (unit 1)
+    (in_bom yes) (on_board yes) (dnp no)
+    (property "Reference" "#PWR0146" (at 177.8 151.765 0)
+      (effects (font (size 1.27 1.27)) hide)
+    )
+    (property "Value" "GND" (at 180.8988 151.892 90)
       (effects (font (size 1.27 1.27)) (justify right))
     )
-    (property "Footprint" "" (at 184.15 148.59 0)
-      (effects (font (size 1.27 1.27)) hide)
-    )
-    (property "Datasheet" "" (at 184.15 148.59 0)
+    (property "Footprint" "" (at 184.15 151.765 0)
+      (effects (font (size 1.27 1.27)) hide)
+    )
+    (property "Datasheet" "" (at 184.15 151.765 0)
       (effects (font (size 1.27 1.27)) hide)
     )
@@
     )
   )
-  (symbol (lib_id "Device:Antenna") (at 222.25 123.19 0) (unit 1)
-    (in_bom yes) (on_board yes) (dnp no)
-    (property "Reference" "AE1" (at 224.282 123.4694 0)
-      (effects (font (size 1.27 1.27)) (justify left))
-    )
-    (property "Value" "Antenna" (at 224.282 125.7808 0)
-      (effects (font (size 1.27 1.27)) (justify left))
-    )
-    (property "Footprint" "jeffmakes-footprints:Antenna_TI_DN038" (at 222.25 123.19 0)
-      (effects (font (size 1.27 1.27)) hide)
-    )
-    (property "Datasheet" "~" (at 222.25 123.19 0)
-      (effects (font (size 1.27 1.27)) hide)
-    )
+  (symbol (lib_id "Device:Antenna") (at 227.965 123.19 0) (unit 1)
+    (in_bom yes) (on_board yes) (dnp no)
+    (property "Reference" "AE1" (at 229.997 123.4694 0)
+      (effects (font (size 1.27 1.27)) (justify left))
+    )
+    (property "Value" "Antenna" (at 229.997 125.7808 0)
+      (effects (font (size 1.27 1.27)) (justify left))
+    )
+    (property "Footprint" "jeffmakes-footprints:Antenna_TI_DN038" (at 227.965 123.19 0)
+      (effects (font (size 1.27 1.27)) hide)
+    )
+    (property "Datasheet" "~" (at 227.965 123.19 0)
+      (effects (font (size 1.27 1.27)) hide)
+    )

Commit message: Exclude test pads, graphics, etc., from BOM
Parts:
- AE1, TP34, TP35: now left out of the parts list
Changed lines of the file:
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@@
   )
   (symbol (lib_id "Connector:TestPoint") (at 73.66 68.58 90) (unit 1)
-    (in_bom yes) (on_board yes) (dnp no)
+    (in_bom no) (on_board yes) (dnp no)
     (property "Reference" "TP34" (at 71.12 66.675 90)
       (effects (font (size 1.27 1.27)))
@@
   )
   (symbol (lib_id "Connector:TestPoint") (at 73.66 71.12 90) (unit 1)
-    (in_bom yes) (on_board yes) (dnp no)
+    (in_bom no) (on_board yes) (dnp no)
     (property "Reference" "TP35" (at 71.12 69.215 90)
       (effects (font (size 1.27 1.27)))
@@
   )
   (symbol (lib_id "Device:Antenna") (at 227.965 123.19 0) (unit 1)
-    (in_bom yes) (on_board yes) (dnp no)
+    (in_bom no) (on_board yes) (dnp no)
     (property "Reference" "AE1" (at 229.997 123.4694 0)
       (effects (font (size 1.27 1.27)) (justify left))
