File: r1/src/tr23-badge-r1.kicad_sch (KiCad schematic)
At the start: 58 parts, among them Q1 MMBT3904-TP, Q2 MMBT3904-TP, Q3 MMBT3904-TP, Y1 32.768kHz

Commit message: Assign footprints from jeffmakes-footprints lib
Parts:
- TP1, TP10, TP11, TP12, TP13, TP14, TP15, TP16, TP17, TP18, TP19, TP2, TP20, TP21, TP22, TP23, TP24, TP25, TP26, TP27, TP28, TP29, TP3, TP30, TP31, TP32, TP4, TP5, TP6, TP7, TP8, TP9: footprint jeffmakes-footprints:test-pad-1.4-TH -> jeffmakes_footprints:test-pad-1.4-TH
Changed lines of the file:
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@@
       (effects (font (size 1.27 1.27)) hide)
     )
-    (property "Footprint" "jeffmakes-footprints:test-pad-1.4-TH" (at 52.07 39.37 0)
+    (property "Footprint" "jeffmakes_footprints:test-pad-1.4-TH" (at 52.07 39.37 0)
       (effects (font (size 1.27 1.27)) hide)
     )
@@
       (effects (font (size 1.27 1.27)) hide)
     )
-    (property "Footprint" "jeffmakes-footprints:test-pad-1.4-TH" (at 52.07 44.45 0)
+    (property "Footprint" "jeffmakes_footprints:test-pad-1.4-TH" (at 52.07 44.45 0)
       (effects (font (size 1.27 1.27)) hide)
     )
@@
       (effects (font (size 1.27 1.27)) hide)
     )
-    (property "Footprint" "jeffmakes-footprints:test-pad-1.4-TH" (at 52.07 46.99 0)
+    (property "Footprint" "jeffmakes_footprints:test-pad-1.4-TH" (at 52.07 46.99 0)
       (effects (font (size 1.27 1.27)) hide)
     )
@@
       (effects (font (size 1.27 1.27)) hide)
     )
-    (property "Footprint" "jeffmakes-footprints:test-pad-1.4-TH" (at 52.07 49.53 0)
+    (property "Footprint" "jeffmakes_footprints:test-pad-1.4-TH" (at 52.07 49.53 0)
       (effects (font (size 1.27 1.27)) hide)
     )
@@
       (effects (font (size 1.27 1.27)) hide)
     )
-    (property "Footprint" "jeffmakes-footprints:test-pad-1.4-TH" (at 52.07 52.07 0)
+    (property "Footprint" "jeffmakes_footprints:test-pad-1.4-TH" (at 52.07 52.07 0)
       (effects (font (size 1.27 1.27)) hide)
     )
@@
       (effects (font (size 1.27 1.27)) hide)
     )
-    (property "Footprint" "jeffmakes-footprints:test-pad-1.4-TH" (at 52.07 62.23 0)
+    (property "Footprint" "jeffmakes_footprints:test-pad-1.4-TH" (at 52.07 62.23 0)
       (effects (font (size 1.27 1.27)) hide)
     )
@@
       (effects (font (size 1.27 1.27)) hide)
     )
-    (property "Footprint" "jeffmakes-footprints:test-pad-1.4-TH" (at 52.07 64.77 0)
+    (property "Footprint" "jeffmakes_footprints:test-pad-1.4-TH" (at 52.07 64.77 0)
       (effects (font (size 1.27 1.27)) hide)
     )
@@
       (effects (font (size 1.27 1.27)) hide)
     )
-    (property "Footprint" "jeffmakes-footprints:test-pad-1.4-TH" (at 52.07 67.31 0)
+    (property "Footprint" "jeffmakes_footprints:test-pad-1.4-TH" (at 52.07 67.31 0)
       (effects (font (size 1.27 1.27)) hide)
     )
@@
       (effects (font (size 1.27 1.27)) hide)
     )
-    (property "Footprint" "jeffmakes-footprints:test-pad-1.4-TH" (at 52.07 69.85 0)
+    (property "Footprint" "jeffmakes_footprints:test-pad-1.4-TH" (at 52.07 69.85 0)
       (effects (font (size 1.27 1.27)) hide)
     )
@@
       (effects (font (size 1.27 1.27)) hide)
     )
-    (property "Footprint" "jeffmakes-footprints:test-pad-1.4-TH" (at 52.07 74.93 0)
+    (property "Footprint" "jeffmakes_footprints:test-pad-1.4-TH" (at 52.07 74.93 0)
       (effects (font (size 1.27 1.27)) hide)
     )
@@
       (effects (font (size 1.27 1.27)) hide)
     )
-    (property "Footprint" "jeffmakes-footprints:test-pad-1.4-TH" (at 110.49 67.31 0)
+    (property "Footprint" "jeffmakes_footprints:test-pad-1.4-TH" (at 110.49 67.31 0)
       (effects (font (size 1.27 1.27)) hide)
     )
@@
       (effects (font (size 1.27 1.27)) hide)
     )
-    (property "Footprint" "jeffmakes-footprints:test-pad-1.4-TH" (at 110.49 72.39 0)
+    (property "Footprint" "jeffmakes_footprints:test-pad-1.4-TH" (at 110.49 72.39 0)
       (effects (font (size 1.27 1.27)) hide)
     )
@@
       (effects (font (size 1.27 1.27)) hide)
     )
-    (property "Footprint" "jeffmakes-footprints:test-pad-1.4-TH" (at 110.49 74.93 0)
+    (property "Footprint" "jeffmakes_footprints:test-pad-1.4-TH" (at 110.49 74.93 0)
       (effects (font (size 1.27 1.27)) hide)
     )
@@
       (effects (font (size 1.27 1.27)) hide)
     )
-    (property "Footprint" "jeffmakes-footprints:test-pad-1.4-TH" (at 110.49 80.01 0)
+    (property "Footprint" "jeffmakes_footprints:test-pad-1.4-TH" (at 110.49 80.01 0)
       (effects (font (size 1.27 1.27)) hide)
     )
@@
       (effects (font (size 1.27 1.27)) hide)
     )
-    (property "Footprint" "jeffmakes-footprints:test-pad-1.4-TH" (at 110.49 82.55 0)
+    (property "Footprint" "jeffmakes_footprints:test-pad-1.4-TH" (at 110.49 82.55 0)
       (effects (font (size 1.27 1.27)) hide)
     )
@@
       (effects (font (size 1.27 1.27)) hide)
     )
-    (property "Footprint" "jeffmakes-footprints:test-pad-1.4-TH" (at 110.49 85.09 0)
+    (property "Footprint" "jeffmakes_footprints:test-pad-1.4-TH" (at 110.49 85.09 0)
       (effects (font (size 1.27 1.27)) hide)
     )
@@
       (effects (font (size 1.27 1.27)) hide)
     )
-    (property "Footprint" "jeffmakes-footprints:test-pad-1.4-TH" (at 110.49 87.63 0)
+    (property "Footprint" "jeffmakes_footprints:test-pad-1.4-TH" (at 110.49 87.63 0)
       (effects (font (size 1.27 1.27)) hide)
     )
@@
       (effects (font (size 1.27 1.27)) hide)
     )
-    (property "Footprint" "jeffmakes-footprints:test-pad-1.4-TH" (at 52.07 83.82 0)
+    (property "Footprint" "jeffmakes_footprints:test-pad-1.4-TH" (at 52.07 83.82 0)
       (effects (font (size 1.27 1.27)) hide)
     )
@@
       (effects (font (size 1.27 1.27)) hide)
     )
-    (property "Footprint" "jeffmakes-footprints:test-pad-1.4-TH" (at 52.07 54.61 0)
+    (property "Footprint" "jeffmakes_footprints:test-pad-1.4-TH" (at 52.07 54.61 0)
       (effects (font (size 1.27 1.27)) hide)
     )
@@
       (effects (font (size 1.27 1.27)) hide)
     )
-    (property "Footprint" "jeffmakes-footprints:test-pad-1.4-TH" (at 52.07 57.15 0)
+    (property "Footprint" "jeffmakes_footprints:test-pad-1.4-TH" (at 52.07 57.15 0)
       (effects (font (size 1.27 1.27)) hide)
     )
@@
       (effects (font (size 1.27 1.27)) hide)
     )
-    (property "Footprint" "jeffmakes-footprints:test-pad-1.4-TH" (at 52.07 59.69 0)
+    (property "Footprint" "jeffmakes_footprints:test-pad-1.4-TH" (at 52.07 59.69 0)
       (effects (font (size 1.27 1.27)) hide)
     )
@@
       (effects (font (size 1.27 1.27)) hide)
     )
-    (property "Footprint" "jeffmakes-footprints:test-pad-1.4-TH" (at 52.07 72.39 0)
+    (property "Footprint" "jeffmakes_footprints:test-pad-1.4-TH" (at 52.07 72.39 0)
       (effects (font (size 1.27 1.27)) hide)
     )
@@
       (effects (font (size 1.27 1.27)) hide)
     )
-    (property "Footprint" "jeffmakes-footprints:test-pad-1.4-TH" (at 52.07 77.47 0)
+    (property "Footprint" "jeffmakes_footprints:test-pad-1.4-TH" (at 52.07 77.47 0)
       (effects (font (size 1.27 1.27)) hide)
     )
@@
       (effects (font (size 1.27 1.27)) hide)
     )
-    (property "Footprint" "jeffmakes-footprints:test-pad-1.4-TH" (at 110.49 54.61 0)
+    (property "Footprint" "jeffmakes_footprints:test-pad-1.4-TH" (at 110.49 54.61 0)
       (effects (font (size 1.27 1.27)) hide)
     )
@@
       (effects (font (size 1.27 1.27)) hide)
     )
-    (property "Footprint" "jeffmakes-footprints:test-pad-1.4-TH" (at 110.49 57.15 0)
+    (property "Footprint" "jeffmakes_footprints:test-pad-1.4-TH" (at 110.49 57.15 0)
       (effects (font (size 1.27 1.27)) hide)
     )
@@
       (effects (font (size 1.27 1.27)) hide)
     )
-    (property "Footprint" "jeffmakes-footprints:test-pad-1.4-TH" (at 110.49 59.69 0)
+    (property "Footprint" "jeffmakes_footprints:test-pad-1.4-TH" (at 110.49 59.69 0)
       (effects (font (size 1.27 1.27)) hide)
     )
@@
       (effects (font (size 1.27 1.27)) hide)
     )
-    (property "Footprint" "jeffmakes-footprints:test-pad-1.4-TH" (at 110.49 62.23 0)
+    (property "Footprint" "jeffmakes_footprints:test-pad-1.4-TH" (at 110.49 62.23 0)
       (effects (font (size 1.27 1.27)) hide)
     )
@@
       (effects (font (size 1.27 1.27)) hide)
     )
-    (property "Footprint" "jeffmakes-footprints:test-pad-1.4-TH" (at 110.49 64.77 0)
+    (property "Footprint" "jeffmakes_footprints:test-pad-1.4-TH" (at 110.49 64.77 0)
       (effects (font (size 1.27 1.27)) hide)
     )
@@
       (effects (font (size 1.27 1.27)) hide)
     )
-    (property "Footprint" "jeffmakes-footprints:test-pad-1.4-TH" (at 110.49 69.85 0)
+    (property "Footprint" "jeffmakes_footprints:test-pad-1.4-TH" (at 110.49 69.85 0)
       (effects (font (size 1.27 1.27)) hide)
     )
@@
       (effects (font (size 1.27 1.27)) hide)
     )
-    (property "Footprint" "jeffmakes-footprints:test-pad-1.4-TH" (at 110.49 77.47 0)
+    (property "Footprint" "jeffmakes_footprints:test-pad-1.4-TH" (at 110.49 77.47 0)
       (effects (font (size 1.27 1.27)) hide)
     )
@@
       (effects (font (size 1.27 1.27)) hide)
     )
-    (property "Footprint" "jeffmakes-footprints:test-pad-1.4-TH" (at 127 36.83 0)
+    (property "Footprint" "jeffmakes_footprints:test-pad-1.4-TH" (at 127 36.83 0)
       (effects (font (size 1.27 1.27)) hide)
     )
@@
       (effects (font (size 1.27 1.27)) hide)
     )
-    (property "Footprint" "jeffmakes-footprints:test-pad-1.4-TH" (at 52.07 81.28 0)
-      (effects (font (size 1.27 1.27)) hide)
-    )
+    (property "Footprint" "jeffmakes_footprints:test-pad-1.4-TH" (at 52.07 81.28 0)
+      (effects (font (size 1.27 1.27)) hide)
+    )

Commit message: Assign footprints
Parts:
- A1: footprint XCVR_ESP32-WROVER-I -> jeffmakes_footprints:ESP32-WROVER-I
- Q1, Q2, Q3: footprint digikey-footprints:SOT-23-3 -> Package_TO_SOT_SMD:SOT-23
- S1, S2: footprint digikey-footprints:Switch_Tactile_SMD_6x6mm_PTS645 -> Button_Switch_SMD:SW_SPST_PTS645
Changed lines of the file:
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@@
       (effects (font (size 1.27 1.27)))
     )
-    (property "Footprint" "XCVR_ESP32-WROVER-I" (at 81.28 62.23 0)
+    (property "Footprint" "jeffmakes_footprints:ESP32-WROVER-I" (at 81.28 62.23 0)
       (effects (font (size 1.27 1.27)) (justify left bottom) hide)
     )
@@
       (effects (font (size 1.524 1.524)) (justify left))
     )
-    (property "Footprint" "digikey-footprints:SOT-23-3" (at 60.96 113.03 0)
+    (property "Footprint" "Package_TO_SOT_SMD:SOT-23" (at 60.96 113.03 0)
       (effects (font (size 1.27 1.27)) hide)
     )
@@
       (effects (font (size 1.524 1.524)) (justify left))
     )
-    (property "Footprint" "digikey-footprints:SOT-23-3" (at 60.96 134.62 0)
+    (property "Footprint" "Package_TO_SOT_SMD:SOT-23" (at 60.96 134.62 0)
       (effects (font (size 1.27 1.27)) hide)
     )
@@
       (effects (font (size 1.524 1.524)) (justify left))
     )
-    (property "Footprint" "digikey-footprints:SOT-23-3" (at 60.96 152.4 0)
+    (property "Footprint" "Package_TO_SOT_SMD:SOT-23" (at 60.96 152.4 0)
       (effects (font (size 1.27 1.27)) hide)
     )
@@
       (effects (font (size 1.524 1.524)) (justify right))
     )
-    (property "Footprint" "digikey-footprints:Switch_Tactile_SMD_6x6mm_PTS645" (at 123.19 132.08 0)
+    (property "Footprint" "Button_Switch_SMD:SW_SPST_PTS645" (at 123.19 132.08 0)
       (effects (font (size 1.27 1.27)) hide)
     )
@@
       (effects (font (size 1.524 1.524)) (justify right))
     )
-    (property "Footprint" "digikey-footprints:Switch_Tactile_SMD_6x6mm_PTS645" (at 134.62 177.8 0)
-      (effects (font (size 1.27 1.27)) hide)
-    )
+    (property "Footprint" "Button_Switch_SMD:SW_SPST_PTS645" (at 134.62 177.8 0)
+      (effects (font (size 1.27 1.27)) hide)
+    )
