File: r1/src/tr23-badge-r1.kicad_sch (KiCad schematic)
At the start: 58 parts, among them Q1 MMBT3904-TP, Q2 MMBT3904-TP, Q3 MMBT3904-TP, Y1 32.768kHz

Commit message: ERC pass. Schematic complete.
Parts:
- added GRAPHIC1: ~, tr23-svg2sz:tr23-r1-svg2sz, symbol j_Display:Display_dummy
- A1: footprint jeffmakes_footprints:ESP32-WROVER-I -> jeffmakes-footprints:ESP32-WROVER-I
- S1, S2: symbol Switch:SW_MEC_5E -> Switch:SW_Push
- TP1, TP10, TP11, TP12, TP13, TP14, TP15, TP16, TP17, TP18, TP19, TP2, TP20, TP21, TP22, TP23, TP24, TP25, TP26, TP27, TP28, TP29, TP3, TP30, TP31, TP32, TP4, TP5, TP6, TP7, TP8, TP9: footprint jeffmakes_footprints:test-pad-1.4-TH -> jeffmakes-footprints:test-pad-1.4-TH
Connections:
- net IO0 is gone; now on net ~{RESET}: Q2.3 (C)
- net GND: now also S1.2, S2.2; no longer S1.4 (A), S2.4 (A)
- no-connect marks 4 -> 0

Commit message: Assign more net classes. Set RF 50ohm width with coplanar ground-backed calculation
Parts:
- added GRAPHIC1: ~, jeffmakes-footprints:Batt_375080_1500mAh, symbol j_Display:Display_dummy
- TP1, TP10, TP11, TP12, TP13, TP14, TP15, TP16, TP17, TP18, TP19, TP2, TP20, TP21, TP22, TP23, TP24, TP25, TP26, TP27, TP28, TP29, TP3, TP30, TP31, TP32, TP4, TP5, TP6, TP7, TP8, TP9: footprint jeffmakes-footprints:test-pad-1.4-TH -> jeffmakes-footprints:test-pad-D1.4
- TP33: footprint TestPoint:TestPoint_Pad_D1.0mm -> jeffmakes-footprints:test-pad-D1.4
Other:
- moved on the sheet: GRAPHIC1

Commit message: Change tact button footprint
Parts:
- S1, S2: footprint Button_Switch_SMD:SW_SPST_PTS645 -> jeffmakes-footprints:SW_SPST_TACT-6x6-no-silk
Changed lines of the file:
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@@
       (effects (font (size 1.524 1.524)) (justify right))
     )
-    (property "Footprint" "Button_Switch_SMD:SW_SPST_PTS645" (at 123.19 132.08 0)
+    (property "Footprint" "jeffmakes-footprints:SW_SPST_TACT-6x6-no-silk" (at 123.19 132.08 0)
       (effects (font (size 1.27 1.27)) hide)
     )
@@
       (effects (font (size 1.524 1.524)) (justify right))
     )
-    (property "Footprint" "Button_Switch_SMD:SW_SPST_PTS645" (at 134.62 177.8 0)
+    (property "Footprint" "jeffmakes-footprints:SW_SPST_TACT-6x6-no-silk" (at 134.62 177.8 0)
       (effects (font (size 1.27 1.27)) hide)
     )

Commit message: Exclude test pads, graphics, etc., from BOM
Parts:
- FID1, FID2, FID3, FID4, FID5, FID6, GRAPHIC1, TP1, TP10, TP11, TP12, TP13, TP14, TP15, TP16, TP17, TP18, TP19, TP2, TP20, TP21, TP22, TP23, TP24, TP25, TP26, TP27, TP28, TP29, TP3, TP30, TP31, TP32, TP33, TP4, TP5, TP6, TP7, TP8, TP9: now left out of the parts list
