File: r1/src/_io_expander.kicad_sch (KiCad schematic)
At the start: 7 parts, among them U4 PCA9555

Commit message: Update all symbols
Parts:
- S6: footprint jeffmakes-footprints:SW_JS1400BFQ-arrows -> SW_JS1400BFQ
Changed lines of the file:
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@@
       (effects (font (size 1.27 1.27)))
     )
-    (property "Footprint" "jeffmakes-footprints:SW_JS1400BFQ-arrows" (at 166.37 97.79 0)
+    (property "Footprint" "SW_JS1400BFQ" (at 166.37 97.79 0)
       (effects (font (size 1.27 1.27)) (justify left bottom) hide)
     )

Commit message: Remove unnecessary module-level labels
Connections:
- net BTN_INT renamed INT
Other:
- note added: "Address = 0x20"
- note removed: "Address = 0x77"
Changed lines of the file:
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@@
     (stroke (width 0) (type default))
   )
-  (wire (pts (xy 52.07 73.66) (xy 40.64 73.66))
+  (wire (pts (xy 52.07 73.66) (xy 44.45 73.66))
     (stroke (width 0) (type default))
   )
@@
     (stroke (width 0) (type default))
   )
-  (wire (pts (xy 63.5 68.58) (xy 40.64 68.58))
+  (wire (pts (xy 63.5 68.58) (xy 44.45 68.58))
     (stroke (width 0) (type default))
   )
@@
     (stroke (width 0) (type default))
   )
-  (wire (pts (xy 63.5 71.12) (xy 40.64 71.12))
+  (wire (pts (xy 63.5 71.12) (xy 44.45 71.12))
     (stroke (width 0) (type default))
   )
@@
     (stroke (width 0) (type default))
   )
-  (text "Address = 0x77\n" (at 81.28 97.79 0)
+  (text "Address = 0x20" (at 81.28 97.79 0)
     (effects (font (size 1.27 1.27)) (justify left bottom))
   )
-  (label "JOY_D" (at 187.96 97.79 180)
+  (label "JOY_D" (at 187.96 97.79 180) (fields_autoplaced)
     (effects (font (size 1.27 1.27)) (justify right bottom))
   )
-  (label "BTN_START" (at 130.81 31.75 270)
+  (label "BTN_START" (at 130.81 31.75 270) (fields_autoplaced)
     (effects (font (size 1.27 1.27)) (justify right bottom))
   )
-  (label "JOY_C" (at 142.24 97.79 0)
+  (label "JOY_C" (at 142.24 97.79 0) (fields_autoplaced)
     (effects (font (size 1.27 1.27)) (justify left bottom))
   )
-  (label "JOY_B" (at 104.14 76.2 180)
+  (label "JOY_B" (at 104.14 76.2 180) (fields_autoplaced)
     (effects (font (size 1.27 1.27)) (justify right bottom))
   )
-  (label "JOY_B" (at 187.96 92.71 180)
+  (label "JOY_B" (at 187.96 92.71 180) (fields_autoplaced)
     (effects (font (size 1.27 1.27)) (justify right bottom))
   )
-  (label "JOY_D" (at 104.14 81.28 180)
+  (label "JOY_D" (at 104.14 81.28 180) (fields_autoplaced)
     (effects (font (size 1.27 1.27)) (justify right bottom))
   )
-  (label "JOY_PUSH" (at 142.24 95.25 0)
+  (label "JOY_PUSH" (at 142.24 95.25 0) (fields_autoplaced)
     (effects (font (size 1.27 1.27)) (justify left bottom))
   )
-  (label "BTN_A" (at 104.14 86.36 180)
+  (label "BTN_A" (at 104.14 86.36 180) (fields_autoplaced)
     (effects (font (size 1.27 1.27)) (justify right bottom))
   )
-  (label "SDA" (at 40.64 71.12 0)
+  (label "JOY_A" (at 142.24 92.71 0) (fields_autoplaced)
     (effects (font (size 1.27 1.27)) (justify left bottom))
   )
-  (label "JOY_A" (at 142.24 92.71 0)
-    (effects (font (size 1.27 1.27)) (justify left bottom))
-  )
-  (label "BTN_INT" (at 40.64 73.66 0)
-    (effects (font (size 1.27 1.27)) (justify left bottom))
-  )
-  (label "BTN_B" (at 104.14 88.9 180)
+  (label "BTN_B" (at 104.14 88.9 180) (fields_autoplaced)
     (effects (font (size 1.27 1.27)) (justify right bottom))
   )
-  (label "BTN_A" (at 168.91 31.75 270)
+  (label "BTN_A" (at 168.91 31.75 270) (fields_autoplaced)
     (effects (font (size 1.27 1.27)) (justify right bottom))
   )
-  (label "BTN_B" (at 207.01 31.75 270)
+  (label "BTN_B" (at 207.01 31.75 270) (fields_autoplaced)
     (effects (font (size 1.27 1.27)) (justify right bottom))
   )
-  (label "JOY_C" (at 104.14 78.74 180)
+  (label "JOY_C" (at 104.14 78.74 180) (fields_autoplaced)
     (effects (font (size 1.27 1.27)) (justify right bottom))
   )
-  (label "JOY_A" (at 104.14 73.66 180)
+  (label "JOY_A" (at 104.14 73.66 180) (fields_autoplaced)
     (effects (font (size 1.27 1.27)) (justify right bottom))
   )
-  (label "JOY_PUSH" (at 104.14 83.82 180)
+  (label "JOY_PUSH" (at 104.14 83.82 180) (fields_autoplaced)
     (effects (font (size 1.27 1.27)) (justify right bottom))
   )
-  (label "BTN_START" (at 104.14 91.44 180)
+  (label "BTN_START" (at 104.14 91.44 180) (fields_autoplaced)
     (effects (font (size 1.27 1.27)) (justify right bottom))
   )
-  (label "SCL" (at 40.64 68.58 0)
-    (effects (font (size 1.27 1.27)) (justify left bottom))
-  )
-  (hierarchical_label "P1_3" (shape bidirectional) (at 100.33 59.69 0)
+  (hierarchical_label "P1_3" (shape bidirectional) (at 100.33 59.69 0) (fields_autoplaced)
     (effects (font (size 1.27 1.27)) (justify left))
   )
-  (hierarchical_label "P1_6" (shape bidirectional) (at 100.33 67.31 0)
+  (hierarchical_label "P1_6" (shape bidirectional) (at 100.33 67.31 0) (fields_autoplaced)
     (effects (font (size 1.27 1.27)) (justify left))
   )
-  (hierarchical_label "P1_1" (shape bidirectional) (at 100.33 54.61 0)
+  (hierarchical_label "P1_1" (shape bidirectional) (at 100.33 54.61 0) (fields_autoplaced)
     (effects (font (size 1.27 1.27)) (justify left))
   )
-  (hierarchical_label "BTN_INT" (shape output) (at 40.64 73.66 180)
+  (hierarchical_label "INT" (shape output) (at 44.45 73.66 180) (fields_autoplaced)
     (effects (font (size 1.27 1.27)) (justify right))
   )
-  (hierarchical_label "SCL" (shape input) (at 40.64 68.58 180)
+  (hierarchical_label "SCL" (shape input) (at 44.45 68.58 180) (fields_autoplaced)
     (effects (font (size 1.27 1.27)) (justify right))
   )
-  (hierarchical_label "SDA" (shape bidirectional) (at 40.64 71.12 180)
+  (hierarchical_label "SDA" (shape bidirectional) (at 44.45 71.12 180) (fields_autoplaced)
     (effects (font (size 1.27 1.27)) (justify right))
   )
-  (hierarchical_label "P1_2" (shape bidirectional) (at 100.33 57.15 0)
+  (hierarchical_label "P1_2" (shape bidirectional) (at 100.33 57.15 0) (fields_autoplaced)
     (effects (font (size 1.27 1.27)) (justify left))
   )
-  (hierarchical_label "P1_7" (shape bidirectional) (at 100.33 69.85 0)
+  (hierarchical_label "P1_7" (shape bidirectional) (at 100.33 69.85 0) (fields_autoplaced)
     (effects (font (size 1.27 1.27)) (justify left))
   )
-  (hierarchical_label "P1_5" (shape bidirectional) (at 100.33 64.77 0)
+  (hierarchical_label "P1_5" (shape bidirectional) (at 100.33 64.77 0) (fields_autoplaced)
     (effects (font (size 1.27 1.27)) (justify left))
   )
-  (hierarchical_label "P1_0" (shape bidirectional) (at 100.33 52.07 0)
+  (hierarchical_label "P1_0" (shape bidirectional) (at 100.33 52.07 0) (fields_autoplaced)
     (effects (font (size 1.27 1.27)) (justify left))
   )
-  (hierarchical_label "P1_4" (shape bidirectional) (at 100.33 62.23 0)
+  (hierarchical_label "P1_4" (shape bidirectional) (at 100.33 62.23 0) (fields_autoplaced)
     (effects (font (size 1.27 1.27)) (justify left))
   )

Commit message: Assign MPN's and LCSC part numbers
Parts:
- S4, S5, S7: value PTS645SM43SMTR92_LFS -> Orange?; MPN PTS645SM43SMTR92 LFS -> (none)
- S6: LCSC (none) -> C145899; MPN (none) -> K1-5202UA-03
- U4: value PCA9555 -> PCA9555PW; LCSC (none) -> C128392; MPN (none) -> PCA9555PW
Changed lines of the file:
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@@
       (effects (font (size 1.27 1.27)))
     )
-    (property "Value" "PCA9555" (at 83.82 48.26 0)
+    (property "Value" "PCA9555PW" (at 83.82 48.26 0)
       (effects (font (size 1.27 1.27)))
     )
@@
     )
     (property "Datasheet" "" (at 77.47 71.12 0)
+      (effects (font (size 1.27 1.27)) hide)
+    )
+    (property "MPN" "PCA9555PW" (at 77.47 71.12 0)
+      (effects (font (size 1.27 1.27)) hide)
+    )
+    (property "LCSC" "C128392" (at 77.47 71.12 0)
       (effects (font (size 1.27 1.27)) hide)
     )
@@
       (effects (font (size 1.27 1.27)) (justify left bottom) hide)
     )
+    (property "LCSC" "C145899" (at 166.37 97.79 0)
+      (effects (font (size 1.27 1.27)) hide)
+    )
+    (property "MPN" "K1-5202UA-03" (at 166.37 97.79 0)
+      (effects (font (size 1.27 1.27)) hide)
+    )
     (pin "1")
     (pin "2")
@@
       (effects (font (size 1.524 1.524)) (justify right))
     )
-    (property "Value" "PTS645SM43SMTR92_LFS" (at 132.08 50.8 90)
+    (property "Value" "Orange?" (at 132.08 50.8 90)
       (effects (font (size 1.524 1.524)) (justify right))
     )
@@
       (effects (font (size 1.524 1.524)) (justify left) hide)
     )
-    (property "MPN" "PTS645SM43SMTR92 LFS" (at 118.11 44.45 0)
+    (property "MPN" "" (at 118.11 44.45 0)
       (effects (font (size 1.524 1.524)) (justify left) hide)
     )
@@
       (effects (font (size 1.524 1.524)) (justify right))
     )
-    (property "Value" "PTS645SM43SMTR92_LFS" (at 170.18 50.9524 90)
+    (property "Value" "Orange?" (at 170.18 50.9524 90)
       (effects (font (size 1.524 1.524)) (justify right))
     )
@@
       (effects (font (size 1.524 1.524)) (justify left) hide)
     )
-    (property "MPN" "PTS645SM43SMTR92 LFS" (at 156.21 44.45 0)
+    (property "MPN" "" (at 156.21 44.45 0)
       (effects (font (size 1.524 1.524)) (justify left) hide)
     )
@@
       (effects (font (size 1.524 1.524)) (justify right))
     )
-    (property "Value" "PTS645SM43SMTR92_LFS" (at 210.5914 50.8762 90)
+    (property "Value" "Orange?" (at 210.5914 50.8762 90)
       (effects (font (size 1.524 1.524)) (justify right))
     )
@@
       (effects (font (size 1.524 1.524)) (justify left) hide)
     )
-    (property "MPN" "PTS645SM43SMTR92 LFS" (at 194.31 44.45 0)
-      (effects (font (size 1.524 1.524)) (justify left) hide)
-    )
+    (property "MPN" "" (at 194.31 44.45 0)
+      (effects (font (size 1.524 1.524)) (justify left) hide)
+    )

Commit message: Assign manufacturers
Parts:
- S6: value JS1400BFQ -> K1-5202UA-03; Manufacturer (none) -> HRO
- U4: Manufacturer (none) -> Texas Instruments
Changed lines of the file:
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@@
+      (effects (font (size 1.27 1.27)) hide)
+    )
+    (property "Manufacturer" "Texas Instruments" (at 77.47 71.12 0)
       (effects (font (size 1.27 1.27)) hide)
     )
@@
       (effects (font (size 1.27 1.27)))
     )
-    (property "Value" " JS1400BFQ" (at 166.37 88.2904 0)
+    (property "Value" "K1-5202UA-03" (at 166.37 88.2904 0)
       (effects (font (size 1.27 1.27)))
     )
@@
       (effects (font (size 1.27 1.27)) hide)
     )
+    (property "Manufacturer" "HRO" (at 166.37 97.79 0)
+      (effects (font (size 1.27 1.27)) hide)
+    )

Commit message: Reannotate component refs
Parts:
- renumbered C75 to C38, R19 to R26, S6 to S5, S5 to S6, U4 to U6
Changed lines of the file:
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@@
   (symbol (lib_id "power:GND") (at 168.91 57.15 0) (unit 1)
     (in_bom yes) (on_board yes) (dnp no)
-    (property "Reference" "#PWR044" (at 168.91 63.5 0)
+    (property "Reference" "#PWR087" (at 168.91 63.5 0)
       (effects (font (size 1.27 1.27)) hide)
     )
@@
       (project "tr23-badge-r1"
         (path "/ab725fe7-4504-40ef-b6af-82d065d00fb6/00000000-0000-0000-0000-00005e0e2ea7"
-          (reference "#PWR044") (unit 1)
+          (reference "#PWR087") (unit 1)
         )
       )
@@
   (symbol (lib_id "power:GND") (at 77.47 96.52 0) (unit 1)
     (in_bom yes) (on_board yes) (dnp no)
-    (property "Reference" "#PWR040" (at 77.47 102.87 0)
+    (property "Reference" "#PWR083" (at 77.47 102.87 0)
       (effects (font (size 1.27 1.27)) hide)
     )
@@
       (project "tr23-badge-r1"
         (path "/ab725fe7-4504-40ef-b6af-82d065d00fb6/00000000-0000-0000-0000-00005e0e2ea7"
-          (reference "#PWR040") (unit 1)
+          (reference "#PWR083") (unit 1)
         )
       )
@@
   (symbol (lib_id "power:GND") (at 130.81 57.15 0) (unit 1)
     (in_bom yes) (on_board yes) (dnp no)
-    (property "Reference" "#PWR042" (at 130.81 63.5 0)
+    (property "Reference" "#PWR085" (at 130.81 63.5 0)
       (effects (font (size 1.27 1.27)) hide)
     )
@@
       (project "tr23-badge-r1"
         (path "/ab725fe7-4504-40ef-b6af-82d065d00fb6/00000000-0000-0000-0000-00005e0e2ea7"
-          (reference "#PWR042") (unit 1)
+          (reference "#PWR085") (unit 1)
         )
       )
@@
   (symbol (lib_id "Device:R") (at 52.07 62.23 0) (mirror y) (unit 1)
     (in_bom yes) (on_board yes) (dnp no)
-    (property "Reference" "R19" (at 50.292 61.0616 0)
+    (property "Reference" "R26" (at 50.292 61.0616 0)
       (effects (font (size 1.27 1.27)) (justify left))
     )
@@
       (project "tr23-badge-r1"
         (path "/ab725fe7-4504-40ef-b6af-82d065d00fb6/00000000-0000-0000-0000-00005e0e2ea7"
-          (reference "R19") (unit 1)
+          (reference "R26") (unit 1)
         )
       )
@@
   (symbol (lib_id "power:GND") (at 93.98 41.91 0) (unit 1)
     (in_bom yes) (on_board yes) (dnp no)
-    (property "Reference" "#PWR041" (at 93.98 48.26 0)
+    (property "Reference" "#PWR084" (at 93.98 48.26 0)
       (effects (font (size 1.27 1.27)) hide)
     )
@@
       (project "tr23-badge-r1"
         (path "/ab725fe7-4504-40ef-b6af-82d065d00fb6/00000000-0000-0000-0000-00005e0e2ea7"
-          (reference "#PWR041") (unit 1)
+          (reference "#PWR084") (unit 1)
         )
       )
@@
   (symbol (lib_id "Device:C") (at 93.98 38.1 0) (mirror y) (unit 1)
     (in_bom yes) (on_board yes) (dnp no)
-    (property "Reference" "C75" (at 91.059 36.9316 0)
+    (property "Reference" "C38" (at 91.059 36.9316 0)
       (effects (font (size 1.27 1.27)) (justify left))
     )
@@
       (project "tr23-badge-r1"
         (path "/ab725fe7-4504-40ef-b6af-82d065d00fb6/00000000-0000-0000-0000-00005e0e2ea7"
-          (reference "C75") (unit 1)
+          (reference "C38") (unit 1)
         )
       )
@@
   (symbol (lib_id "power:GND") (at 156.21 105.41 0) (unit 1)
     (in_bom yes) (on_board yes) (dnp no)
-    (property "Reference" "#PWR0122" (at 156.21 111.76 0)
+    (property "Reference" "#PWR086" (at 156.21 111.76 0)
       (effects (font (size 1.27 1.27)) hide)
     )
@@
       (project "tr23-badge-r1"
         (path "/ab725fe7-4504-40ef-b6af-82d065d00fb6/00000000-0000-0000-0000-00005e0e2ea7"
-          (reference "#PWR0122") (unit 1)
+          (reference "#PWR086") (unit 1)
         )
       )
@@
   (symbol (lib_id "j_Interface_Expansion:PCA9555") (at 77.47 71.12 0) (unit 1)
     (in_bom yes) (on_board yes) (dnp no)
-    (property "Reference" "U4" (at 81.28 45.72 0)
+    (property "Reference" "U6" (at 81.28 45.72 0)
       (effects (font (size 1.27 1.27)))
     )
@@
       (project "tr23-badge-r1"
         (path "/ab725fe7-4504-40ef-b6af-82d065d00fb6/00000000-0000-0000-0000-00005e0e2ea7"
-          (reference "U4") (unit 1)
+          (reference "U6") (unit 1)
         )
       )
@@
   (symbol (lib_id "power:GND") (at 59.69 58.42 270) (unit 1)
     (in_bom yes) (on_board yes) (dnp no)
-    (property "Reference" "#PWR0115" (at 53.34 58.42 0)
+    (property "Reference" "#PWR081" (at 53.34 58.42 0)
       (effects (font (size 1.27 1.27)) hide)
     )
@@
       (project "tr23-badge-r1"
         (path "/ab725fe7-4504-40ef-b6af-82d065d00fb6/00000000-0000-0000-0000-00005e0e2ea7"
-          (reference "#PWR0115") (unit 1)
+          (reference "#PWR081") (unit 1)
         )
       )
@@
   (symbol (lib_id "power:GND") (at 176.53 95.25 90) (unit 1)
     (in_bom yes) (on_board yes) (dnp no)
-    (property "Reference" "#PWR0116" (at 182.88 95.25 0)
+    (property "Reference" "#PWR088" (at 182.88 95.25 0)
       (effects (font (size 1.27 1.27)) hide)
     )
@@
       (project "tr23-badge-r1"
         (path "/ab725fe7-4504-40ef-b6af-82d065d00fb6/00000000-0000-0000-0000-00005e0e2ea7"
-          (reference "#PWR0116") (unit 1)
+          (reference "#PWR088") (unit 1)
         )
       )
@@
   (symbol (lib_id "j_Switch:TMHU13-B") (at 166.37 97.79 0) (unit 1)
     (in_bom yes) (on_board yes) (dnp no)
-    (property "Reference" "S6" (at 166.37 85.979 0)
+    (property "Reference" "S5" (at 166.37 85.979 0)
       (effects (font (size 1.27 1.27)))
     )
@@
       (project "tr23-badge-r1"
         (path "/ab725fe7-4504-40ef-b6af-82d065d00fb6/00000000-0000-0000-0000-00005e0e2ea7"
-          (reference "S6") (unit 1)
+          (reference "S5") (unit 1)
         )
         (path "/ab725fe7-4504-40ef-b6af-82d065d00fb6"
@@
   (symbol (lib_id "Switch:SW_MEC_5E") (at 168.91 49.53 90) (unit 1)
     (in_bom yes) (on_board yes) (dnp no)
-    (property "Reference" "S5" (at 170.18 48.26 90)
+    (property "Reference" "S6" (at 170.18 48.26 90)
       (effects (font (size 1.524 1.524)) (justify right))
     )
@@
       (project "tr23-badge-r1"
         (path "/ab725fe7-4504-40ef-b6af-82d065d00fb6/00000000-0000-0000-0000-00005e0e2ea7"
-          (reference "S5") (unit 1)
+          (reference "S6") (unit 1)
         )
         (path "/ab725fe7-4504-40ef-b6af-82d065d00fb6"
@@
   (symbol (lib_id "power:+3.3V") (at 52.07 54.61 0) (unit 1)
     (in_bom yes) (on_board yes) (dnp no)
-    (property "Reference" "#PWR038" (at 52.07 58.42 0)
+    (property "Reference" "#PWR080" (at 52.07 58.42 0)
       (effects (font (size 1.27 1.27)) hide)
     )
@@
       (project "tr23-badge-r1"
         (path "/ab725fe7-4504-40ef-b6af-82d065d00fb6/00000000-0000-0000-0000-00005e0e2ea7"
-          (reference "#PWR038") (unit 1)
+          (reference "#PWR080") (unit 1)
         )
       )
@@
   (symbol (lib_id "power:+3.3V") (at 77.47 30.48 0) (unit 1)
     (in_bom yes) (on_board yes) (dnp no)
-    (property "Reference" "#PWR039" (at 77.47 34.29 0)
+    (property "Reference" "#PWR082" (at 77.47 34.29 0)
       (effects (font (size 1.27 1.27)) hide)
     )
@@
       (project "tr23-badge-r1"
         (path "/ab725fe7-4504-40ef-b6af-82d065d00fb6/00000000-0000-0000-0000-00005e0e2ea7"
-          (reference "#PWR039") (unit 1)
+          (reference "#PWR082") (unit 1)
         )
       )
@@
   (symbol (lib_id "power:GND") (at 207.01 57.15 0) (unit 1)
     (in_bom yes) (on_board yes) (dnp no)
-    (property "Reference" "#PWR048" (at 207.01 63.5 0)
+    (property "Reference" "#PWR089" (at 207.01 63.5 0)
       (effects (font (size 1.27 1.27)) hide)
     )
@@
       (project "tr23-badge-r1"
         (path "/ab725fe7-4504-40ef-b6af-82d065d00fb6/00000000-0000-0000-0000-00005e0e2ea7"
-          (reference "#PWR048") (unit 1)
-        )
-      )
+          (reference "#PWR089") (unit 1)
+        )
+      )

Commit message: Assign footprints from jeffmakes-footprints lib
Parts:
- S5: footprint SW_JS1400BFQ -> jeffmakes_footprints:SW_JS1400BFQ-arrows
Changed lines of the file:
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@@
       (effects (font (size 1.27 1.27)))
     )
-    (property "Footprint" "SW_JS1400BFQ" (at 166.37 97.79 0)
+    (property "Footprint" "jeffmakes_footprints:SW_JS1400BFQ-arrows" (at 166.37 97.79 0)
       (effects (font (size 1.27 1.27)) (justify left bottom) hide)
     )

Commit message: Assign footprints
Parts:
- S4, S6, S7: footprint digikey-footprints:Switch_Tactile_SMD_6x6mm_PTS645 -> Button_Switch_SMD:SW_SPST_PTS645
Changed lines of the file:
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@@
       (effects (font (size 1.524 1.524)) (justify right))
     )
-    (property "Footprint" "digikey-footprints:Switch_Tactile_SMD_6x6mm_PTS645" (at 123.19 49.53 0)
+    (property "Footprint" "Button_Switch_SMD:SW_SPST_PTS645" (at 123.19 49.53 0)
       (effects (font (size 1.27 1.27)) hide)
     )
@@
       (effects (font (size 1.524 1.524)) (justify right))
     )
-    (property "Footprint" "digikey-footprints:Switch_Tactile_SMD_6x6mm_PTS645" (at 161.29 49.53 0)
+    (property "Footprint" "Button_Switch_SMD:SW_SPST_PTS645" (at 161.29 49.53 0)
       (effects (font (size 1.27 1.27)) hide)
     )
@@
       (effects (font (size 1.524 1.524)) (justify right))
     )
-    (property "Footprint" "digikey-footprints:Switch_Tactile_SMD_6x6mm_PTS645" (at 199.39 49.53 0)
+    (property "Footprint" "Button_Switch_SMD:SW_SPST_PTS645" (at 199.39 49.53 0)
       (effects (font (size 1.27 1.27)) hide)
     )
