File: r1/src/_io_expander.kicad_sch (KiCad schematic)
At the start: 7 parts, among them U6 PCA9555PW

Commit message: Switch 5-way nav switch footprint.
Parts:
- S5: footprint jeffmakes-footprints:SW_JS1400BFQ-arrows -> jeffmakes-footprints:SW_JS1400BFQ
Changed lines of the file:
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@@
       (effects (font (size 1.27 1.27)))
     )
-    (property "Footprint" "jeffmakes-footprints:SW_JS1400BFQ-arrows" (at 166.37 97.79 0)
+    (property "Footprint" "jeffmakes-footprints:SW_JS1400BFQ" (at 166.37 97.79 0)
       (effects (font (size 1.27 1.27)) (justify left bottom) hide)
     )

Commit message: Change tact button footprint
Parts:
- S4, S6, S7: footprint Button_Switch_SMD:SW_SPST_PTS645 -> jeffmakes-footprints:SW_SPST_TACT-6x6-no-silk
Changed lines of the file:
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@@
       (effects (font (size 1.524 1.524)) (justify right))
     )
-    (property "Footprint" "Button_Switch_SMD:SW_SPST_PTS645" (at 125.73 49.53 0)
+    (property "Footprint" "jeffmakes-footprints:SW_SPST_TACT-6x6-no-silk" (at 125.73 49.53 0)
       (effects (font (size 1.27 1.27)) hide)
     )
@@
       (effects (font (size 1.524 1.524)) (justify right))
     )
-    (property "Footprint" "Button_Switch_SMD:SW_SPST_PTS645" (at 163.83 49.53 0)
+    (property "Footprint" "jeffmakes-footprints:SW_SPST_TACT-6x6-no-silk" (at 163.83 49.53 0)
       (effects (font (size 1.27 1.27)) hide)
     )
@@
       (effects (font (size 1.524 1.524)) (justify right))
     )
-    (property "Footprint" "Button_Switch_SMD:SW_SPST_PTS645" (at 201.93 49.53 0)
+    (property "Footprint" "jeffmakes-footprints:SW_SPST_TACT-6x6-no-silk" (at 201.93 49.53 0)
       (effects (font (size 1.27 1.27)) hide)
     )
