File: tr23-outline-test-r1/src/tr23-outline-test-r1.kicad_pcb (KiCad board)
At the start: 2 copper layers, 111.2 x 142.3 mm, 37 parts

Commit message: Place switches, start routing
Parts:
- removed REF** (x2): PinSocket_2x03_P2.54mm_Through-Board-Mating, jeffmakes-kicad-library:PinSocket_2x03_P2.54mm_Through-Board-Mating
- SW1, SW10, SW11, SW12, SW13, SW14, SW15, SW16, SW17, SW18, SW19, SW2, SW20, SW21, SW22, SW23, SW24, SW25, SW26, SW27, SW28, SW29, SW3, SW30, SW31, SW32, SW33, SW34, SW4, SW5, SW6, SW7, SW8, SW9: renamed from REF**; value SW_SPST_TACT_6x6_REV_MOUNT -> REV_TACT
- turned SW33 to 135 degrees
Connections:
- SW1 pad 1: (no net) -> GND
- SW1 pad 2: (no net) -> GND
- SW1 pad 3: (no net) -> /KEY0
- SW1 pad 4: (no net) -> /KEY0
- SW10 pad 1: (no net) -> GND
- SW10 pad 2: (no net) -> GND
- SW10 pad 3: (no net) -> /KEY10
- SW10 pad 4: (no net) -> /KEY10
- SW11 pad 1: (no net) -> GND
- SW11 pad 2: (no net) -> GND
- SW11 pad 3: (no net) -> /KEY18
- SW11 pad 4: (no net) -> /KEY18
- SW12 pad 1: (no net) -> GND
- SW12 pad 2: (no net) -> GND
- SW12 pad 3: (no net) -> /KEY26
- SW12 pad 4: (no net) -> /KEY26
- SW13 pad 1: (no net) -> GND
- SW13 pad 2: (no net) -> GND
- SW13 pad 3: (no net) -> /KEY3
- SW13 pad 4: (no net) -> /KEY3
- SW14 pad 1: (no net) -> GND
- SW14 pad 2: (no net) -> GND
- SW14 pad 3: (no net) -> /KEY11
- SW14 pad 4: (no net) -> /KEY11
- SW15 pad 1: (no net) -> GND
- SW15 pad 2: (no net) -> GND
- SW15 pad 3: (no net) -> /KEY19
- SW15 pad 4: (no net) -> /KEY19
- SW16 pad 1: (no net) -> GND
- SW16 pad 2: (no net) -> GND
- SW16 pad 3: (no net) -> /KEY27
- SW16 pad 4: (no net) -> /KEY27
- SW17 pad 1: (no net) -> GND
- SW17 pad 2: (no net) -> GND
- SW17 pad 3: (no net) -> /KEY4
- SW17 pad 4: (no net) -> /KEY4
- SW18 pad 1: (no net) -> GND
- SW18 pad 2: (no net) -> GND
- SW18 pad 3: (no net) -> /KEY12
- SW18 pad 4: (no net) -> /KEY12
- SW19 pad 1: (no net) -> GND
- SW19 pad 2: (no net) -> GND
- SW19 pad 3: (no net) -> /KEY20
- SW19 pad 4: (no net) -> /KEY20
- SW2 pad 1: (no net) -> GND
- SW2 pad 2: (no net) -> GND
- SW2 pad 3: (no net) -> /KEY8
- SW2 pad 4: (no net) -> /KEY8
- SW20 pad 1: (no net) -> GND
- SW20 pad 2: (no net) -> GND
- SW20 pad 3: (no net) -> /KEY28
- SW20 pad 4: (no net) -> /KEY28
- SW21 pad 1: (no net) -> GND
- SW21 pad 2: (no net) -> GND
- SW21 pad 3: (no net) -> /KEY5
- SW21 pad 4: (no net) -> /KEY5
- SW22 pad 1: (no net) -> GND
- SW22 pad 2: (no net) -> GND
- SW22 pad 3: (no net) -> /KEY13
- SW22 pad 4: (no net) -> /KEY13
- SW23 pad 1: (no net) -> GND
- SW23 pad 2: (no net) -> GND
- SW23 pad 3: (no net) -> /KEY21
- SW23 pad 4: (no net) -> /KEY21
- SW24 pad 1: (no net) -> GND
- SW24 pad 2: (no net) -> GND
- SW24 pad 3: (no net) -> /KEY29
- SW24 pad 4: (no net) -> /KEY29
- SW25 pad 1: (no net) -> GND
- SW25 pad 2: (no net) -> GND
- SW25 pad 3: (no net) -> /KEY6
- SW25 pad 4: (no net) -> /KEY6
- SW26 pad 1: (no net) -> GND
- SW26 pad 2: (no net) -> GND
- SW26 pad 3: (no net) -> /KEY14
- SW26 pad 4: (no net) -> /KEY14
- SW27 pad 1: (no net) -> GND
- SW27 pad 2: (no net) -> GND
- SW27 pad 3: (no net) -> /KEY22
- SW27 pad 4: (no net) -> /KEY22
- SW28 pad 1: (no net) -> GND
- SW28 pad 2: (no net) -> GND
- SW28 pad 3: (no net) -> /KEY30
- SW28 pad 4: (no net) -> /KEY30
- SW29 pad 1: (no net) -> GND
- SW29 pad 2: (no net) -> GND
- SW29 pad 3: (no net) -> /KEY7
- SW29 pad 4: (no net) -> /KEY7
- SW3 pad 1: (no net) -> GND
- SW3 pad 2: (no net) -> GND
- SW3 pad 3: (no net) -> /KEY16
- SW3 pad 4: (no net) -> /KEY16
- SW30 pad 1: (no net) -> GND
- SW30 pad 2: (no net) -> GND
- SW30 pad 3: (no net) -> /KEY15
- SW30 pad 4: (no net) -> /KEY15
- SW31 pad 1: (no net) -> GND
- SW31 pad 2: (no net) -> GND
- SW31 pad 3: (no net) -> /KEY23
- SW31 pad 4: (no net) -> /KEY23
- SW32 pad 1: (no net) -> GND
- SW32 pad 2: (no net) -> GND
- SW32 pad 3: (no net) -> /KEY31
- SW32 pad 4: (no net) -> /KEY31
- SW33 pad 1: (no net) -> GND
- SW33 pad 2: (no net) -> GND
- SW33 pad 3: (no net) -> /KEY31
- SW33 pad 4: (no net) -> /KEY31
- SW34 pad 1: (no net) -> GND
- SW34 pad 2: (no net) -> GND
- SW34 pad 3: (no net) -> /KEY31
- SW34 pad 4: (no net) -> /KEY31
- SW4 pad 1: (no net) -> GND
- SW4 pad 2: (no net) -> GND
- SW4 pad 3: (no net) -> /KEY24
- SW4 pad 4: (no net) -> /KEY24
- SW5 pad 1: (no net) -> GND
- SW5 pad 2: (no net) -> GND
- SW5 pad 3: (no net) -> /KEY1
- SW5 pad 4: (no net) -> /KEY1
- SW6 pad 1: (no net) -> GND
- SW6 pad 2: (no net) -> GND
- SW6 pad 3: (no net) -> /KEY9
- SW6 pad 4: (no net) -> /KEY9
- SW7 pad 1: (no net) -> GND
- SW7 pad 2: (no net) -> GND
- SW7 pad 3: (no net) -> /KEY17
- SW7 pad 4: (no net) -> /KEY17
- SW8 pad 1: (no net) -> GND
- SW8 pad 2: (no net) -> GND
- SW8 pad 3: (no net) -> /KEY25
- SW8 pad 4: (no net) -> /KEY25
- SW9 pad 1: (no net) -> GND
- SW9 pad 2: (no net) -> GND
- SW9 pad 3: (no net) -> /KEY2
- SW9 pad 4: (no net) -> /KEY2
Routing:
- net /KEY22: track 0.00 -> 40.2 mm
- net /KEY20: track 0.00 -> 31.5 mm
- net /KEY12: track 0.00 -> 31.2 mm
- net /KEY4: track 0.00 -> 30.9 mm
- net /KEY14: track 0.00 -> 29.8 mm
- net /KEY6: track 0.00 -> 28.7 mm
- net /KEY10: track 0.00 -> 19.2 mm
- net /KEY2: track 0.00 -> 18.4 mm
- net /KEY25: track 0.00 -> 15.1 mm
- added copper zone on B.Cu, net GND

Commit message: Update SVG export
Parts:
- added REF**: Z280IT009, jeffmakes-kicad-library:Z280IT009, F.Cu at (-28.6, -56.0)
- added TP1: ~, TestPoint:TestPoint_Pad_D1.5mm, B.Cu at (-62.5, -37.5)
- added TP10: ~, TestPoint:TestPoint_Pad_D1.5mm, B.Cu at (-22.5, -37.5)
- added TP11: ~, TestPoint:TestPoint_Pad_D1.5mm, B.Cu at (17.5, -37.5)
- added TP12: ~, TestPoint:TestPoint_Pad_D1.5mm, B.Cu at (-35.0, -37.5)
- added TP13: ~, TestPoint:TestPoint_Pad_D1.5mm, B.Cu at (0.00, -37.5)
- added TP14: ~, TestPoint:TestPoint_Pad_D1.5mm, B.Cu at (-32.5, -37.5)
- added TP15: ~, TestPoint:TestPoint_Pad_D1.5mm, B.Cu at (2.50, -37.5)
- added TP16: ~, TestPoint:TestPoint_Pad_D1.5mm, B.Cu at (-5.00, -37.5)
- added TP17: ~, TestPoint:TestPoint_Pad_D1.5mm, B.Cu at (-47.5, -37.5)
- added TP18: ~, TestPoint:TestPoint_Pad_D1.5mm, B.Cu at (-12.5, -37.5)
- added TP19: ~, TestPoint:TestPoint_Pad_D1.5mm, B.Cu at (-60.0, -37.5)
- added TP2: ~, TestPoint:TestPoint_Pad_D1.5mm, B.Cu at (-30.0, -37.5)
- added TP20: ~, TestPoint:TestPoint_Pad_D1.5mm, B.Cu at (-27.5, -37.5)
- added TP21: ~, TestPoint:TestPoint_Pad_D1.5mm, B.Cu at (12.5, -37.5)
- added TP22: ~, TestPoint:TestPoint_Pad_D1.5mm, B.Cu at (-25.0, -37.5)
- added TP23: ~, TestPoint:TestPoint_Pad_D1.5mm, B.Cu at (15.0, -37.5)
- added TP24: ~, TestPoint:TestPoint_Pad_D1.5mm, B.Cu at (5.00, -37.5)
- added TP25: ~, TestPoint:TestPoint_Pad_D1.5mm, B.Cu at (-37.5, -37.5)
- added TP26: ~, TestPoint:TestPoint_Pad_D1.5mm, B.Cu at (-2.50, -37.5)
- added TP27: ~, TestPoint:TestPoint_Pad_D1.5mm, B.Cu at (-55.0, -37.5)
- added TP28: ~, TestPoint:TestPoint_Pad_D1.5mm, B.Cu at (-20.0, -37.5)
- added TP29: ~, TestPoint:TestPoint_Pad_D1.5mm, B.Cu at (-52.5, -37.5)
- added TP3: ~, TestPoint:TestPoint_Pad_D1.5mm, B.Cu at (7.50, -37.5)
- added TP30: ~, TestPoint:TestPoint_Pad_D1.5mm, B.Cu at (-17.5, -37.5)
- added TP31: ~, TestPoint:TestPoint_Pad_D1.5mm, B.Cu at (-50.0, -37.5)
- added TP32: ~, TestPoint:TestPoint_Pad_D1.5mm, B.Cu at (-15.0, -37.5)
- added TP33: ~, TestPoint:TestPoint_Pad_D1.5mm, B.Cu at (17.5, -40.0)
- added TP4: ~, TestPoint:TestPoint_Pad_D1.5mm, B.Cu at (-45.0, -37.5)
- added TP5: ~, TestPoint:TestPoint_Pad_D1.5mm, B.Cu at (-10.0, -37.5)
- added TP6: ~, TestPoint:TestPoint_Pad_D1.5mm, B.Cu at (-42.5, -37.5)
- added TP7: ~, TestPoint:TestPoint_Pad_D1.5mm, B.Cu at (-7.50, -37.5)
- added TP8: ~, TestPoint:TestPoint_Pad_D1.5mm, B.Cu at (-40.0, -37.5)
- added TP9: ~, TestPoint:TestPoint_Pad_D1.5mm, B.Cu at (-57.5, -37.5)
Connections:
- SW1 pad 1: GND -> unconnected-(SW1-Pad1)
- SW1 pad 4: /KEY0 -> unconnected-(SW1-A-Pad4)
- SW10 pad 1: GND -> unconnected-(SW10-Pad1)
- SW10 pad 4: /KEY10 -> unconnected-(SW10-A-Pad4)
- SW11 pad 1: GND -> unconnected-(SW11-Pad1)
- SW11 pad 4: /KEY18 -> unconnected-(SW11-A-Pad4)
- SW12 pad 1: GND -> unconnected-(SW12-Pad1)
- SW12 pad 4: /KEY26 -> unconnected-(SW12-A-Pad4)
- SW13 pad 1: GND -> unconnected-(SW13-Pad1)
- SW13 pad 4: /KEY3 -> unconnected-(SW13-A-Pad4)
- SW14 pad 1: GND -> unconnected-(SW14-Pad1)
- SW14 pad 4: /KEY11 -> unconnected-(SW14-A-Pad4)
- SW15 pad 1: GND -> unconnected-(SW15-Pad1)
- SW15 pad 4: /KEY19 -> unconnected-(SW15-A-Pad4)
- SW16 pad 1: GND -> unconnected-(SW16-Pad1)
- SW16 pad 4: /KEY27 -> unconnected-(SW16-A-Pad4)
- SW17 pad 1: GND -> unconnected-(SW17-Pad1)
- SW17 pad 4: /KEY4 -> unconnected-(SW17-A-Pad4)
- SW18 pad 1: GND -> unconnected-(SW18-Pad1)
- SW18 pad 4: /KEY12 -> unconnected-(SW18-A-Pad4)
- SW19 pad 1: GND -> unconnected-(SW19-Pad1)
- SW19 pad 4: /KEY20 -> unconnected-(SW19-A-Pad4)
- SW2 pad 1: GND -> unconnected-(SW2-Pad1)
- SW2 pad 4: /KEY8 -> unconnected-(SW2-A-Pad4)
- SW20 pad 1: GND -> unconnected-(SW20-Pad1)
- SW20 pad 4: /KEY28 -> unconnected-(SW20-A-Pad4)
- SW21 pad 1: GND -> unconnected-(SW21-Pad1)
- SW21 pad 4: /KEY5 -> unconnected-(SW21-A-Pad4)
- SW22 pad 1: GND -> unconnected-(SW22-Pad1)
- SW22 pad 4: /KEY13 -> unconnected-(SW22-A-Pad4)
- SW23 pad 1: GND -> unconnected-(SW23-Pad1)
- SW23 pad 4: /KEY21 -> unconnected-(SW23-A-Pad4)
- SW24 pad 1: GND -> unconnected-(SW24-Pad1)
- SW24 pad 4: /KEY29 -> unconnected-(SW24-A-Pad4)
- SW25 pad 1: GND -> unconnected-(SW25-Pad1)
- SW25 pad 4: /KEY6 -> unconnected-(SW25-A-Pad4)
- SW26 pad 1: GND -> unconnected-(SW26-Pad1)
- SW26 pad 4: /KEY14 -> unconnected-(SW26-A-Pad4)
- SW27 pad 1: GND -> unconnected-(SW27-Pad1)
- SW27 pad 4: /KEY22 -> unconnected-(SW27-A-Pad4)
- SW28 pad 1: GND -> unconnected-(SW28-Pad1)
- SW28 pad 4: /KEY30 -> unconnected-(SW28-A-Pad4)
- SW29 pad 1: GND -> unconnected-(SW29-Pad1)
- SW29 pad 4: /KEY7 -> unconnected-(SW29-A-Pad4)
- SW3 pad 1: GND -> unconnected-(SW3-Pad1)
- SW3 pad 4: /KEY16 -> unconnected-(SW3-A-Pad4)
- SW30 pad 1: GND -> unconnected-(SW30-Pad1)
- SW30 pad 4: /KEY15 -> unconnected-(SW30-A-Pad4)
- SW31 pad 1: GND -> unconnected-(SW31-Pad1)
- SW31 pad 4: /KEY23 -> unconnected-(SW31-A-Pad4)
- SW32 pad 1: GND -> unconnected-(SW32-Pad1)
- SW32 pad 4: /KEY31 -> unconnected-(SW32-A-Pad4)
- SW33 pad 1: GND -> unconnected-(SW33-Pad1)
- SW33 pad 4: /KEY31 -> unconnected-(SW33-A-Pad4)
- SW34 pad 1: GND -> unconnected-(SW34-Pad1)
- SW34 pad 4: /KEY31 -> unconnected-(SW34-A-Pad4)
- SW4 pad 1: GND -> unconnected-(SW4-Pad1)
- SW4 pad 4: /KEY24 -> unconnected-(SW4-A-Pad4)
- SW5 pad 1: GND -> unconnected-(SW5-Pad1)
- SW5 pad 4: /KEY1 -> unconnected-(SW5-A-Pad4)
- SW6 pad 1: GND -> unconnected-(SW6-Pad1)
- SW6 pad 4: /KEY9 -> unconnected-(SW6-A-Pad4)
- SW7 pad 1: GND -> unconnected-(SW7-Pad1)
- SW7 pad 4: /KEY17 -> unconnected-(SW7-A-Pad4)
- SW8 pad 1: GND -> unconnected-(SW8-Pad1)
- SW8 pad 4: /KEY25 -> unconnected-(SW8-A-Pad4)
- SW9 pad 1: GND -> unconnected-(SW9-Pad1)
- SW9 pad 4: /KEY2 -> unconnected-(SW9-A-Pad4)
Routing:
- net /KEY31: track 0.00 -> 70.6 mm
- net /KEY15: track 0.00 -> 49.2 mm
- net /KEY23: track 0.00 -> 49.0 mm
- net /KEY7: track 0.00 -> 48.5 mm
- net /KEY30: track 0.00 -> 48.4 mm
- net /KEY29: track 0.00 -> 33.3 mm
- net /KEY28: track 0.00 -> 32.8 mm
- net /KEY21: track 0.00 -> 32.6 mm
- net /KEY13: track 0.00 -> 32.4 mm
- net /KEY5: track 0.00 -> 32.4 mm
- net /KEY27: track 0.00 -> 26.8 mm
- net /KEY26: track 0.00 -> 26.2 mm
- net /KEY19: track 0.00 -> 26.2 mm
- net /KEY3: track 0.00 -> 25.8 mm
- net /KEY18: track 0.00 -> 25.4 mm
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Other:
- outline, holes or cut-outs redrawn
- board text added: "tr23-outline-test-r1 2023-03-10 Monad"
