File: tr23-outline-test-r1/src/tr23-outline-test-r1.kicad_pcb (KiCad board)
At the start: 2 copper layers, 111.2 x 142.3 mm, 69 parts, among them SW1 REV_TACT, SW10 REV_TACT, SW11 REV_TACT, SW12 REV_TACT, SW13 REV_TACT, SW14 REV_TACT, SW15 REV_TACT, SW16 REV_TACT, SW17 REV_TACT, SW18 REV_TACT, SW19 REV_TACT, SW2 REV_TACT, SW20 REV_TACT, SW21 REV_TACT, SW22 REV_TACT, SW23 REV_TACT, SW24 REV_TACT, SW25 REV_TACT, SW26 REV_TACT, SW27 REV_TACT, SW28 REV_TACT, SW29 REV_TACT, SW3 REV_TACT, SW30 REV_TACT, SW31 REV_TACT, SW32 REV_TACT, SW33 REV_TACT, SW34 REV_TACT, SW4 REV_TACT, SW5 REV_TACT, SW6 REV_TACT, SW7 REV_TACT, SW8 REV_TACT, SW9 REV_TACT

Commit message: Lock buttons
Parts:
- renumbered REF** to disp-1

Commit message: Tweak logo position
Parts:
- added J1: Conn_02x03_Counter_Clockwise, jeffmakes-kicad-library:PinSocket_2x03_P2.54mm_Through-Board-Mating, B.Cu at (-25.4, 18.0)
- added S1: TMHU13-B, jeffmakes-kicad-library:SW_JS1400BFQ, F.Cu at (-68.5, -45.9)
- added SW35: SW_MEC_5E, jeffmakes-kicad-library:SW_SPST_TACT-6x6-no-silk, F.Cu at (17.5, -59.4)
- added SW36: SW_MEC_5E, jeffmakes-kicad-library:SW_SPST_TACT-6x6-no-silk, F.Cu at (17.5, -45.9)
- added SW37: SW_MEC_5E, jeffmakes-kicad-library:SW_SPST_TACT-6x6-no-silk, F.Cu at (-68.5, -59.4)
- DISP1: renamed from disp-1; value Z280IT009 -> Z280IT008
- GRAPHIC1: renamed from Ref**; value Val** -> ~
Other:
- outline, holes or cut-outs redrawn
