File: r2/src/_micro_sd.kicad_sch (KiCad schematic)
At the start: 6 parts, among them J7 TF-15x15

Commit message: Set title block contents
Other:
- company: (none) -> Monad Gottfried Ltd. 2023
- title: (none) -> Troopers 23 Badge
Changed lines of the file:
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@@
 (kicad_sch (version 20230409) (generator eeschema)
   (paper "A4")
+  (title_block
+    (title "Troopers 23 Badge")
+    (rev "r2")
+    (company "Monad Gottfried Ltd. 2023")
+    (comment 1 "for ERNW Enno Rey Netzwerke GmbH")
+  )
   (junction (at 144.78 76.2) (diameter 0) (color 0 0 0 0)
   )
