File: r2/src/_shitty_addon.kicad_sch (KiCad schematic)
At the start: 6 parts, among them J6 2x03-socket-2.54-through-board

Commit message: Set title block contents
Other:
- company: (none) -> Monad Gottfried Ltd. 2023
- title: (none) -> Troopers 23 Badge
Changed lines of the file:
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@@
 (kicad_sch (version 20230409) (generator eeschema)
   (paper "A4")
+  (title_block
+    (title "Troopers 23 Badge")
+    (rev "r2")
+    (company "Monad Gottfried Ltd. 2023")
+    (comment 1 "for ERNW Enno Rey Netzwerke GmbH")
+  )
   (junction (at 153.67 119.38) (diameter 0) (color 0 0 0 0)
   )
