File: r2/src/_usb.kicad_sch (KiCad schematic)
At the start: 14 parts, among them J2 TYPE-C3, J3 USB-A-10mm-flangeless, U3 CP2102N-A01-GQFN24

Commit message: Set title block contents
Other:
- company: (none) -> Monad Gottfried Ltd. 2023
- title: (none) -> Troopers 23 Badge
Changed lines of the file:
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@@
 (kicad_sch (version 20230409) (generator eeschema)
   (paper "A4")
+  (title_block
+    (title "Troopers 23 Badge")
+    (rev "r2")
+    (company "Monad Gottfried Ltd. 2023")
+    (comment 1 "for ERNW Enno Rey Netzwerke GmbH")
+  )
   (junction (at 95.25 78.74) (diameter 0) (color 0 0 0 0)
   )
