File: r2/src/tr23-badge-r2.kicad_sch (KiCad schematic)
At the start: 61 parts, among them Q1 MMBT3904-TP, Q2 MMBT3904-TP, Q3 MMBT3904-TP, Y1 32.768kHz

Commit message: Set title block contents
Other:
- company: (none) -> Monad Gottfried Ltd. 2023
- title: (none) -> Troopers 23 Badge
Changed lines of the file:
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@@
 (kicad_sch (version 20230409) (generator eeschema)
   (paper "A4")
+  (title_block
+    (title "Troopers 23 Badge")
+    (rev "r2")
+    (company "Monad Gottfried Ltd. 2023")
+    (comment 1 "for ERNW Enno Rey Netzwerke GmbH")
+  )
   (junction (at 128.27 168.91) (diameter 0) (color 0 0 0 0)
   )
